File: testpcb.kicad_pcb (KiCad board)
At the start: 2 copper layers, 52 parts, among them SW1 SW_Push, U1 ATmega16U4-AU, Y1 16MHz

Commit message: ulozenie git
Parts:
- D1, D10, D11, D12, D13, D14, D15, D16, D17, D2, D3, D4, D5, D6, D7, D8, D9: moved to B.Cu
- R1, R2, R3, R4, R5, R6: footprint Resistor_SMD:R_0815_2038Metric -> Resistor_SMD:R_0805_2012Metric
- moved U1 149.7 mm to (292.1, -14.3)
- moved C4 120.6 mm to (287.3, -4.61), turned to 90 degrees
- moved D11 120.4 mm to (295.3, 29.4), turned to 90 degrees
- moved C3 118.5 mm to (295.3, -4.61), turned to 270 degrees
- moved D6 118.3 mm to (275.4, 10.4), turned to 90 degrees
- moved R1 117.4 mm to (281.0, -19.1), turned to 90 degrees
- moved D15 117.1 mm to (313.5, 10.4), turned to 90 degrees
- moved C2 115.2 mm to (271.5, -4.61), turned to 90 degrees
- moved USB1 113.4 mm to (253.2, -25.4), turned to 180 degrees
- moved D12 111.0 mm to (294.5, 49.3), turned to 90 degrees
- moved D10 107.8 mm to (295.3, 10.4), turned to 90 degrees
- moved D14 107.6 mm to (294.5, 86.6), turned to 90 degrees
- moved R2 107.4 mm to (281.0, -15.7), turned to 90 degrees
- moved D13 107.3 mm to (294.5, 67.5), turned to 90 degrees
- moved R4 106.2 mm to (300.8, -14.4), turned to 90 degrees
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
Commit message: DONE
Parts:
- C1, C2, C3, C4, C5, C6, C7, F1, R1, R2, R3, R4, R5, R6, U1, USB1, Y1: moved to B.Cu
- moved R6 110.8 mm to (360.7, -8.19)
- moved R5 106.1 mm to (358.4, -8.19)
- moved USB1 104.5 mm to (357.5, -20.2), turned to 0 degrees
- moved F1 99.5 mm to (355.1, -8.15)
- moved C5 80.7 mm to (345.6, 0.59)
- moved SW1 75.5 mm to (301.9, -7.10), turned to 90 degrees
- moved C1 74.4 mm to (342.5, 0.59)
- moved C2 68.0 mm to (339.3, 0.59)
- moved D1 62.2 mm to (318.4, 15.4)
- moved D10 62.2 mm to (357.3, 15.4)
- moved D11 62.2 mm to (357.3, 34.4)
- moved D12 62.2 mm to (356.5, 54.3)
- moved D13 62.2 mm to (356.5, 72.5)
- moved D14 62.2 mm to (356.5, 91.6)
- moved D15 62.2 mm to (375.5, 15.4)
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Connections:
- USB1 pad 11: Net-(USB1-Pad11) -> VCC
- USB1 pad 12: Net-(USB1-Pad12) -> GND
- USB1 pad 13: Net-(USB1-Pad13) -> GND
Routing:
- net COL0: track 0.00 -> 80.1 mm
- net GND: track 0.00 -> 77.9 mm
- net COL2: track 0.00 -> 76.2 mm
- net +5V: track 0.00 -> 75.8 mm
- net COL3: track 0.00 -> 73.6 mm
- net COL1: track 0.00 -> 57.2 mm
- net ROW0: track 0.00 -> 57.1 mm
- net ROW3: track 0.00 -> 47.4 mm
- net ROW1: track 0.00 -> 44.0 mm
- net ROW2: track 0.00 -> 38.1 mm
- net Net-(R3-Pad2): track 0.00 -> 33.3 mm, vias 0 -> 1
- net D-: track 0.00 -> 32.7 mm
- net D+: track 0.00 -> 32.5 mm, vias 0 -> 2
- net ROW4: track 0.00 -> 28.6 mm
- net VCC: track 0.00 -> 11.5 mm, vias 0 -> 2
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- added copper zone on B.Cu, net GND
- added copper zone on F.Cu, net GND
Other:
- board outline added: 90 x 130 mm

Commit message: jakies poprawki kolejne
Parts:
- moved D3 0.28 mm to (318.1, 54.3)
- moved D2 0.26 mm to (317.9, 34.4)
Routing:
- net Net-(D3-Pad2): track 9.61 -> 8.41 mm
- net Net-(D8-Pad2): track 9.58 -> 8.61 mm
- net Net-(D2-Pad2): track 8.46 -> 7.57 mm
- net Net-(D12-Pad2): track 9.55 -> 8.67 mm

Commit message: polaczone switche / wizualne poprawki tracerow
Parts:
- moved C7 6.30 mm to (334.6, -7.00)
- moved R1 6.30 mm to (334.7, -12.4)
- moved R2 6.30 mm to (334.6, -9.95)
- moved D11 0.88 mm to (356.4, 34.4)
- moved D10 0.53 mm to (356.8, 15.3)
Connections:
- U1 pad 25: Net-(U1-Pad25) -> COL3
- U1 pad 26: Net-(U1-Pad26) -> COL2
- U1 pad 27: Net-(U1-Pad27) -> COL1
- U1 pad 28: Net-(U1-Pad28) -> COL0
- U1 pad 36: Net-(U1-Pad36) -> ROW0
- U1 pad 37: Net-(U1-Pad37) -> ROW1
- U1 pad 38: Net-(U1-Pad38) -> ROW2
- U1 pad 39: Net-(U1-Pad39) -> ROW3
- U1 pad 40: Net-(U1-Pad40) -> ROW4
Routing:
- net ROW4: track 28.6 -> 173.1 mm
- net ROW3: track 47.4 -> 164.5 mm
- net ROW2: track 38.1 -> 136.3 mm
- net ROW1: track 44.0 -> 120.7 mm
- net COL3: track 73.6 -> 136.9 mm
- net ROW0: track 57.1 -> 112.1 mm
- net COL2: track 76.2 -> 122.1 mm
- net COL1: track 57.2 -> 85.5 mm
- net COL0: track 80.1 -> 104.6 mm
- net D-: track 32.7 -> 25.8 mm
- net Net-(R1-Pad1): track 3.44 -> 9.80 mm
- net Net-(R2-Pad1): track 3.40 -> 9.68 mm
- net Net-(C7-Pad1): track 3.97 -> 10.2 mm
- net GND: track 77.9 -> 83.5 mm
- net D+: track 32.5 -> 27.5 mm
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
Commit message: gowno
Routing:
- net GND: track 83.5 -> 112.2 mm, vias 0 -> 3
- net ROW0: track 112.1 -> 108.3 mm, vias 0 -> 2
- net Net-(R3-Pad2): track 33.3 -> 34.5 mm
- added copper zone on F.Cu, net (none)
- removed copper zone on F.Cu, net GND

Commit message: naprawione coppery
Routing:
- added copper zone on F.Cu, net GND
- removed copper zone on F.Cu, net (none)

Commit message: gowno
Parts:
- MX16, MX17, MX5: footprint MX_Only:MXOnly-2U -> MX_Only:MXOnly-2U-ReversedStabilizers
- moved D14 4.13 mm to (356.4, 87.5)
- moved D12 3.93 mm to (356.4, 50.4)
- moved D11 1.95 mm to (355.9, 36.3)
- moved D13 1.73 mm to (355.8, 74.1)
Routing:
- net GND: track 112.2 -> 101.4 mm, vias 3 -> 18
- net ROW3: track 164.5 -> 171.9 mm
- net ROW1: track 120.7 -> 124.8 mm
- net ROW4: track 173.1 -> 175.7 mm
- net Net-(D12-Pad2): track 8.67 -> 6.64 mm
- net D-: track 25.8 -> 27.7 mm
- net Net-(D14-Pad2): track 7.97 -> 6.22 mm
- net ROW2: track 136.3 -> 137.9 mm
- net Net-(D11-Pad2): track 7.87 -> 8.50 mm
- net COL0: vias 0 -> 1
Other:
- board size 90 x 130 mm -> 83.1 x 130 mm

Commit message: poprawki
Parts:
- moved C2 3.85 mm to (339.2, -3.26)
- moved C5 3.85 mm to (345.6, -3.26)
- moved C6 3.85 mm to (336.1, -3.26)
- moved C1 3.85 mm to (342.4, -3.26)
