File: testpcb.kicad_pcb (KiCad board)
At the start: 2 copper layers, 83.1 x 130 mm, 52 parts, among them SW1 SW_Push, U1 ATmega16U4-AU, Y1 16MHz

Commit message: mounting holes
Parts:
- added H1: MountingHole, MountingHole:MountingHole_2.1mm, F.Cu at (380.9, -11.4)
- added H2: MountingHole, MountingHole:MountingHole_2.1mm, F.Cu at (308.4, -11.4)
- added H3: MountingHole, MountingHole:MountingHole_2.1mm, F.Cu at (308.4, -131.7)
- added H4: MountingHole, MountingHole:MountingHole_2.1mm, F.Cu at (380.9, -131.4)
- added J1: AVR-ISP-6, random-keyboard-parts:Reset_Pretty-Mask, F.Cu at (338.2, -121.7)
- MX16, MX17, MX5: footprint MX_Only:MXOnly-2U-ReversedStabilizers -> MX_Only:MXOnly-2U
- moved C7 123.9 mm to (341.8, -130.7), turned to 90 degrees
- moved R2 120.8 mm to (338.9, -130.7), turned to 90 degrees
- moved R1 118.3 mm to (336.4, -130.7), turned to 90 degrees
- moved C3 116.7 mm to (322.0, -115.9)
- moved C4 116.7 mm to (330.0, -115.9)
- moved D1 116.7 mm to (324.9, -101.1)
- moved D10 116.7 mm to (363.3, -101.2)
- moved D11 116.7 mm to (362.5, -80.2)
- moved D12 116.7 mm to (363.0, -66.2)
- moved D13 116.7 mm to (362.3, -42.4)
- moved D14 116.7 mm to (363.0, -29.1)
- moved D15 116.7 mm to (382.1, -101.1)
- moved D16 116.7 mm to (369.4, -81.3)
- moved D17 116.7 mm to (373.3, -44.0)
- moved D2 116.7 mm to (324.4, -82.1)
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Connections:
- net Net-(R3-Pad2) renamed RESET
- U1 pad 10: Net-(U1-Pad10) -> MOSI
- U1 pad 11: Net-(U1-Pad11) -> MISO
- U1 pad 9: Net-(U1-Pad9) -> SCK
Routing:
- net GND: track 101.4 -> 83.6 mm, vias 18 -> 19
- net +5V: track 76.8 -> 87.2 mm
- net MOSI: track 0.00 -> 9.85 mm, vias 0 -> 1
- net MISO: track 0.00 -> 7.15 mm
- net SCK: track 0.00 -> 6.71 mm, vias 0 -> 1
- net D-: track 27.7 -> 33.7 mm
- net D+: track 27.5 -> 33.3 mm
- net RESET: track 34.5 -> 38.2 mm
- net Net-(C7-Pad1): track 10.2 -> 12.6 mm
- net ROW0: track 108.3 -> 107.5 mm
- net COL0: track 104.6 -> 105.2 mm
- net Net-(D13-Pad2): track 8.12 -> 8.68 mm
